File: pcb/sensor/kicad/eu_sensor_flex.kicad_pcb (KiCad board)
At the start: 2 copper layers, 171.3 x 30.4 mm, 10 parts, among them J1 CN2 mate (TBD), U1 SHT45

Commit message: Smaller plate, flex ramps and tape points, battery-free tongue on the sensor flex, back cover hooks
- Plate 72 x 132, 5 V contact in the corner, band groove, microphone below the band, two-layer
  sensor flex (D-47)
- Ramps over the flex slopes; tape geometry and tape renders (render_tape.py, D-48)
- Battery-free tongue moved from the 5 V jumper to the sensor flex: under the trim's tab and strip,
  under the floor insert, which hangs from the strip; EU tongue under its floor insert (D-49)
- Back cover: bottom latch 2.9 mm from the edge, end-section snap hooks, notch for the run under
  the GND block; plate clips kept for PETG
Routing:
- net GND: track 99.5 -> 107.2 mm
Other:
- outline, holes or cut-outs redrawn
