File: pcb/sensor/kicad/riser_board.kicad_pcb (KiCad board)
At the start: 2 copper layers, 14 x 12 mm, 4 parts, among them J1 +5V pin, J2 GND pin, P1 +5V post, P2 GND post

Commit message: v0.5: back cover ends, mains spacing 3.0 mm, NA fuse separation, labels, bare renders (D-101..D-106)
- D-101: back cover shell gauges (R15..R20.9); the stadium end is confirmed
- D-102: mains spacing 3.0 mm on high-CTI FR4 (MAINS_GAP, NA and EU)
- D-103: back cover end walls 1.40 mm, inside 0.2 mm longer (BC_END_WALL)
- D-104: NA wiring board: any two mains nets 3.0 mm apart, L_F re-routed
  F1.2 -> RV1.1, L_SW vias below F1, L_SW pour up towards the rocker;
  EU mains board checked, unchanged
- D-105: rocker silkscreen "E-Switch RA412C1100 or Marquardt 1802.2504",
  EU 5 V socket part on its label; bare 3D renders for every board
- D-106: version v0.5; v0.4 fab packs, PCBWay packs and renders removed
Other:
- board text added: "RISER v0.5"
- board text removed: "RISER v0.4"
Changed lines of the file:
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@@
+		)
+	)
+	(footprint "sensor:Harwin_P70-2200045"
+		(layer "F.Cu")
+		(at 113.2 108.9)
+		(descr "Harwin P70-2200045 SMT spring pin with peg, pad 2.2 mm, hole 1.2 mm, https://content.harwin.com/asset/7e702b12-8f84-42b5-9282-d7e22f3466f3/DRG-02624-Technical-Drawing-Datasheet-P70-220-pdf.pdf")
+		(tags "spring pin pogo")
+		(property "Reference" "J1"
+			(at 0 0 0)
+			(layer "F.SilkS")
+			(hide yes)
+			(effects
+				(font
+					(size 1 1)
+					(thickness 0.15)
+				)
+			)
+		)
+		(property "Value" "+5V pin"
+			(at 0 0 0)
+			(layer "F.Fab")
+			(hide yes)
+			(effects
+				(font
+					(size 1 1)
+					(thickness 0.15)
+				)
+			)
+		)
+		(property "Datasheet" ""
+			(at 0 0 0)
+			(layer "F.Fab")
+			(hide yes)
+			(effects
+				(font
+					(size 1.27 1.27)
+					(thickness 0.15)
+				)
+			)
+		)
+		(property "Description" ""
+			(at 0 0 0)
+			(layer "F.Fab")
+			(hide yes)
+			(effects
+				(font
+					(size 1.27 1.27)
+					(thickness 0.15)
+				)
+			)
+		)
+		(sheetname "Root")
+		(sheetfile "riser_board.kicad_sch")
+		(attr smd)
+		(fp_circle
+			(center 0 0)
+			(end 1.35 0)
+			(stroke
+				(width 0.05)
+				(type solid)
+			)
+			(fill no)
+			(layer "F.CrtYd")
+		)
+		(fp_circle
+			(center 0 0)
+			(end 1 0)
+			(stroke
+				(width 0.1)
+				(type solid)
+			)
+			(fill no)
+			(layer "F.Fab")
+		)
+		(pad "1" thru_hole circle
+			(at 0 0)
+			(size 2.2 2.2)
+			(drill 1.2)
+			(layers "*.Cu" "*.Mask" "F.Paste")
+			(remove_unused_layers no)
+			(net 1 "+5V")
+		)
+		(embedded_fonts no)
+		(model "${KIPRJMOD}/3d/Harwin_P70-2200045.step"
+			(offset
+				(xyz 0 0 0)
+			)
+			(scale
+				(xyz 1 1 1)
+			)
+			(rotate
+				(xyz 0 0 0)
+			)
 		)
 	)
@@
 		(embedded_fonts no)
 	)
-	(footprint "sensor:Harwin_P70-2200045"
-		(layer "F.Cu")
-		(at 113.2 108.9)
-		(descr "Harwin P70-2200045 SMT spring pin with peg, pad 2.2 mm, hole 1.2 mm, https://content.harwin.com/asset/7e702b12-8f84-42b5-9282-d7e22f3466f3/DRG-02624-Technical-Drawing-Datasheet-P70-220-pdf.pdf")
-		(tags "spring pin pogo")
-		(property "Reference" "J1"
-			(at 0 0 0)
-			(layer "F.SilkS")
-			(hide yes)
-			(effects
-				(font
-					(size 1 1)
-					(thickness 0.15)
-				)
-			)
-		)
-		(property "Value" "+5V pin"
-			(at 0 0 0)
-			(layer "F.Fab")
-			(hide yes)
-			(effects
-				(font
-					(size 1 1)
-					(thickness 0.15)
-				)
-			)
-		)
-		(property "Datasheet" ""
-			(at 0 0 0)
-			(layer "F.Fab")
-			(hide yes)
-			(effects
-				(font
-					(size 1.27 1.27)
-					(thickness 0.15)
-				)
-			)
-		)
-		(property "Description" ""
-			(at 0 0 0)
-			(layer "F.Fab")
-			(hide yes)
-			(effects
-				(font
-					(size 1.27 1.27)
-					(thickness 0.15)
-				)
-			)
-		)
-		(sheetname "Root")
-		(sheetfile "riser_board.kicad_sch")
-		(attr smd)
-		(fp_circle
-			(center 0 0)
-			(end 1.35 0)
-			(stroke
-				(width 0.05)
-				(type solid)
-			)
-			(fill no)
-			(layer "F.CrtYd")
-		)
-		(fp_circle
-			(center 0 0)
-			(end 1 0)
-			(stroke
-				(width 0.1)
-				(type solid)
-			)
-			(fill no)
-			(layer "F.Fab")
-		)
-		(pad "1" thru_hole circle
-			(at 0 0)
-			(size 2.2 2.2)
-			(drill 1.2)
-			(layers "*.Cu" "*.Mask" "F.Paste")
-			(remove_unused_layers no)
-			(net 1 "+5V")
-		)
-		(embedded_fonts no)
-		(model "${KIPRJMOD}/3d/Harwin_P70-2200045.step"
-			(offset
-				(xyz 0 0 0)
-			)
-			(scale
-				(xyz 1 1 1)
-			)
-			(rotate
-				(xyz 0 0 0)
-			)
-		)
-	)
 	(footprint "sensor:M2_Post_Pad_D3.8mm"
 		(layer "F.Cu")
@@
 		(layer "Edge.Cuts")
 	)
-	(gr_text "RISER v0.4"
+	(gr_text "RISER v0.5"
 		(at 113.25 111.2 0)
 		(layer "B.SilkS")
@@
 	)
 	(segment
+		(start 116.65 116.5)
+		(end 115.390354 114.209734)
+		(width 1)
+		(layer "F.Cu")
+		(net 2)
+	)
+	(segment
 		(start 114.19 113.5)
 		(end 113.2 113.5)
 		(width 1)
 		(layer "F.Cu")
-		(net 2)
-	)
-	(segment
-		(start 116.65 116.5)
-		(end 115.390354 114.209734)
-		(width 1)
-		(layer "F.Cu")
