File: pcb/sensor/kicad/cover_flex.kicad_sch (KiCad schematic)
At the start: 7 parts, among them J1 S7081-42R +5V, J2 S7081-42R GND, J3 S7081-42R VBAT, J4 S7081-42R GND, U1 TLV75533PDBVR

Commit message: Back cover: snap hooks for the flex, stronger magnet clips, rounded contact posts; #6 countersink and PLATE_Y on the trim
Parts:
- C3, C4: MPN GRM155R61A105KE15D -> CL05A105KP5NNNC; Manufacturer Murata -> Samsung Electro-Mechanics
Changed lines of the file:
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@@
 			)
 		)
-		(property "Manufacturer" "Murata"
+		(property "Manufacturer" "Samsung Electro-Mechanics"
 			(at 238.76 91.44 0)
 			(effects
@@
 			)
 		)
-		(property "MPN" "GRM155R61A105KE15D"
+		(property "MPN" "CL05A105KP5NNNC"
 			(at 238.76 91.44 0)
 			(effects
@@
 			)
 		)
-		(property "Manufacturer" "Murata"
-			(at 35.56 157.48 0)
-			(effects
-				(font
-					(size 1.27 1.27)
-				)
-				(hide yes)
-			)
-		)
-		(property "MPN" "GRM155R61A105KE15D"
-			(at 35.56 157.48 0)
-			(effects
+		(property "Manufacturer" "Samsung Electro-Mechanics"
+			(at 35.56 157.48 0)
+			(effects
+				(font
+					(size 1.27 1.27)
+				)
+				(hide yes)
+			)
+		)
+		(property "MPN" "CL05A105KP5NNNC"
+			(at 35.56 157.48 0)
+			(effects

Commit message: Boards for v0.4: ring board, mic carrier, riser, cover flex, EU cap board, wiring board posts
- Ring board, mic carrier and riser in pcb/sensor/ (D-50, D-60, D-68); carrier and riser fab
  packs; the ring board waits on the MSR-2's CN2 part and map
- Riser 14 x 12 mm, pins above and between the posts; cover flex with the run past the GND
  contact post and a jog from the pad section (D-79)
- EU cap board on the carrier, closed snap windows, wider with the face plate (D-56, D-70,
  D-77, D-78); EU 5 V board pins follow the back cover's pads
- Wiring board: WA-SMSI spacer posts in the 5 V area (SMT, spigot inside the board), J2
- ERC / DRC clean on every board
Parts:
- J1: value S7081-42R +5V -> +5V pin pad; footprint sensor:Harwin_S7081-42R -> sensor:Contact_Pad_D2.6mm; symbol sensor:Conn_01x01 -> sensor:TestPoint; MPN S7081-42R -> (none); Manufacturer Harwin -> (none); now left out of the parts list
- J2: value S7081-42R GND -> GND pin pad; footprint sensor:Harwin_S7081-42R -> sensor:Contact_Pad_D2.6mm; symbol sensor:Conn_01x01 -> sensor:TestPoint; MPN S7081-42R -> (none); Manufacturer Harwin -> (none); now left out of the parts list
Other:
- note added: "Replacement back cover flex (docs/DESIGN.md D-35, D-50): J1 / J2 pads under the plate's spring pins (+5V, GND), U1 3.3 V regulator, J3 / J4 spring fingers on the BILRESA's VBAT plate / GND leaf spring. One bend, single layer."
- note removed: "Replacement back cover flex (docs/DESIGN.md D-35): J1 / J2 spring fingers on the plate's floor pads (+5V, GND), U1 3.3 V regulator, J3 / J4 spring fingers on the BILRESA's VBAT plate / GND leaf spring. One bend, single layer."

Commit message: Mic on the boards, parts audit, rocker second source, CN2 land pattern, back cover fit (D-82..D-90)
- Prototype PCBWay packs for the ring board, EU cap board and cover flex; logos and URL on the
  boards with room for them
- CN2 mate: Molex 55909-2474 on an assumed 51338-2474 (D-82); land pattern from Molex
  SD-55909-003 rev J, B2B from SD-51338-003 rev K (D-89); contact map and pin 1 still open
- Microphone: Knowles SPK0641HT4H-1 + ADAU7002 on the ring board and the EU cap board, the mic
  carrier removed; face plate sound column on a gasket (D-83); C3 KEMET C1206C104J3GACTU C0G
  (D-85)
- Parts rule (active, stocked at DigiKey or Mouser) and audit: F1 3403.0166.11, cover flex 1 uF
  CL05A105KO5NNNC, rocker at Mouser 979-1802.2504 (D-84)
- Rocker: tabs soldered into plated slots accepted (D-86); E-Switch RA412C1100 second source,
  slotted footprint on the wiring board and the EU mains board, solder the rocker after the
  board is screwed down (D-88)
- Back cover: round-over 8.1 x 8.0 from the printed gauges (D-87); four tabs inside the long
  side walls into the housing's slots (D-90); back_gauges_PLA
- make stock / make order-push (pcb/tools/distributors.py): live DigiKey / Mouser stock and
  lifecycle, DigiKey myLists link and Mouser cart; keys from the environment only
- Boards ERC / DRC clean; make check, make eu, make check-renders pass; renders, fab and
  order packs regenerated
Parts:
- C3, C4: MPN CL05A105KP5NNNC -> CL05A105KO5NNNC
Changed lines of the file:
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@@
 			)
 		)
-		(property "Description" "LDO input capacitor, 1 uF 10 V X5R 0402 (TLV755P: >= 1 uF)"
+		(property "Description" "LDO input capacitor, 1 uF 16 V X5R 0402 (TLV755P: >= 1 uF)"
 			(at 238.76 91.44 0)
 			(effects
@@
 			)
 		)
-		(property "MPN" "CL05A105KP5NNNC"
+		(property "MPN" "CL05A105KO5NNNC"
 			(at 238.76 91.44 0)
 			(effects
@@
 			)
 		)
-		(property "Description" "LDO output capacitor, 1 uF 10 V X5R 0402 (TLV755P: >= 1 uF)"
+		(property "Description" "LDO output capacitor, 1 uF 16 V X5R 0402 (TLV755P: >= 1 uF)"
 			(at 35.56 157.48 0)
 			(effects
@@
 			)
 		)
-		(property "MPN" "CL05A105KP5NNNC"
-			(at 35.56 157.48 0)
-			(effects
+		(property "MPN" "CL05A105KO5NNNC"
+			(at 35.56 157.48 0)
+			(effects

Commit message: Flex review fixes, back cover clip, README, Sladdseg, order lists (D-116..D-119)
- D-116: cover flex: 0603 X5R input/output caps, ESD diode TPD1E10B06DYAR,
  0.6 mm bend radius with relief slits, stiffener notch and outlines,
  coverlay expansion, mask-defined pin pads, teardrops, fab notes; the
  cover's snap hooks allow for stiffener adhesive and tolerance
- D-117, D-118: bottom clip catch 3.22 above the floor, tip as far proud of
  the shell as the top clip's
- Battery polarity confirmed on a unit
- README rewritten: three editions, assembly renders, safety and polarity
  warnings, cost for 1 to 10,000 plates, printed parts; detail and board
  renders moved to their docs; the product is named Sladdseg
- EU boards: the ant logo on the other face
- D-119: order lists: one NA plate, one EU plate, a devkit of 5 + 5
Parts:
- added D1: TPD1E10B06DYAR, sensor:D_SOD-523_TI_DYA0002A, symbol sensor:D_TVS
- C3, C4: value 1uF -> 1uF 16V X5R 0603; footprint sensor:C_0402_1005Metric -> sensor:C_0603_1608Metric; MPN CL05A105KO5NNNC -> CL10A105KO8NNNC
Connections:
- net +5V: now also D1.2 (A2)
- net GND: now also D1.1 (A1)
Other:
- title: Smart wall plate - back cover flex -> Sladdseg - back cover flex
Changed lines of the file:
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@@
 	(paper "A4")
 	(title_block
-		(title "Smart wall plate - back cover flex")
+		(title "Sladdseg - back cover flex")
 		(date "2026-10-12")
 		(rev "v0.5")
@@
 			)
 		)
-		(property "Value" "1uF"
+		(property "Value" "1uF 16V X5R 0603"
 			(at 241.76 99.94 0)
 			(effects
@@
 			)
 		)
-		(property "Footprint" "sensor:C_0402_1005Metric"
+		(property "Footprint" "sensor:C_0603_1608Metric"
 			(at 238.76 91.44 0)
 			(effects
@@
 			)
 		)
-		(property "Datasheet" ""
+		(property "Datasheet" "https://product.samsungsem.com/mlcc/CL10A105KO8NNN.do"
 			(at 238.76 91.44 0)
 			(effects
@@
 			)
 		)
-		(property "Description" "LDO input capacitor, 1 uF 16 V X5R 0402 (TLV755P: >= 1 uF)"
+		(property "Description" "LDO input capacitor, 1 uF 16 V X5R 0603: 0.85 uF at 5 V (TLV755P: >= 0.47 uF effective, D-116)"
 			(at 238.76 91.44 0)
 			(effects
@@
 			)
 		)
-		(property "MPN" "CL05A105KO5NNNC"
+		(property "MPN" "CL10A105KO8NNNC"
 			(at 238.76 91.44 0)
 			(effects
@@
 			)
 		)
-		(property "Value" "1uF"
+		(property "Value" "1uF 16V X5R 0603"
 			(at 38.56 165.98 0)
 			(effects
@@
 			)
 		)
-		(property "Footprint" "sensor:C_0402_1005Metric"
+		(property "Footprint" "sensor:C_0603_1608Metric"
 			(at 35.56 157.48 0)
 			(effects
@@
 			)
 		)
-		(property "Datasheet" ""
+		(property "Datasheet" "https://product.samsungsem.com/mlcc/CL10A105KO8NNN.do"
 			(at 35.56 157.48 0)
 			(effects
@@
 			)
 		)
-		(property "Description" "LDO output capacitor, 1 uF 16 V X5R 0402 (TLV755P: >= 1 uF)"
+		(property "Description" "LDO output capacitor, 1 uF 16 V X5R 0603: 0.93 uF at 3.3 V (TLV755P: >= 0.47 uF effective, D-116)"
 			(at 35.56 157.48 0)
 			(effects
@@
 			)
 		)
-		(property "MPN" "CL05A105KO5NNNC"
+		(property "MPN" "CL10A105KO8NNNC"
 			(at 35.56 157.48 0)
 			(effects
@@
 	)
 	(symbol
+		(lib_id "sensor:D_TVS")
+		(at 76.2 157.48 0)
+		(unit 1)
+		(exclude_from_sim no)
+		(in_bom yes)
+		(on_board yes)
+		(dnp no)
+		(property "Reference" "D1"
+			(at 79.2 149.48 0)
+			(effects
+				(font
+					(size 1.27 1.27)
+				)
+				(justify left)
+			)
+		)
+		(property "Value" "TPD1E10B06DYAR"
+			(at 79.2 165.98 0)
+			(effects
+				(font
+					(size 1.27 1.27)
+				)
+				(justify left)
+			)
+		)
+		(property "Footprint" "sensor:D_SOD-523_TI_DYA0002A"
+			(at 76.2 157.48 0)
+			(effects
+				(font
+					(size 1.27 1.27)
+				)
+				(hide yes)
+			)
+		)
+		(property "Datasheet" "https://www.ti.com/lit/ds/symlink/tpd1e10b06.pdf"
+			(at 76.2 157.48 0)
+			(effects
+				(font
+					(size 1.27 1.27)
+				)
+				(hide yes)
+			)
+		)
+		(property "Description" "ESD protection, bidirectional TVS, 5.5 V working, SOD-523: +5V at the exposed pin pads (D-116)"
+			(at 76.2 157.48 0)
+			(effects
+				(font
+					(size 1.27 1.27)
+				)
+				(hide yes)
+			)
+		)
+		(property "Manufacturer" "Texas Instruments"
+			(at 76.2 157.48 0)
+			(effects
+				(font
+					(size 1.27 1.27)
+				)
+				(hide yes)
+			)
+		)
+		(property "MPN" "TPD1E10B06DYAR"
+			(at 76.2 157.48 0)
+			(effects
+				(font
+					(size 1.27 1.27)
+				)
+				(hide yes)
+			)
+		)
+		(pin "1"
+		)
+		(pin "2"
+		)
+		(instances
+			(project "cover_flex"
+				(path "/b53ed5b7-46c8-5996-a3fb-579e9f592242"
+					(reference "D1")
+					(unit 1)
+				)
+			)
+		)
+	)
+	(symbol
+		(lib_id "sensor:GND")
+		(at 72.39 157.48 0)
+		(unit 1)
+		(exclude_from_sim no)
+		(in_bom no)
+		(on_board no)
+		(dnp no)
+		(property "Reference" "#PWR013"
+			(at 75.39 149.48 0)
+			(effects
+				(font
+					(size 1.27 1.27)
+				)
+				(justify left)
+				(hide yes)
+			)
+		)
+		(property "Value" "GND"
+			(at 75.39 165.98 0)
+			(effects
+				(font
+					(size 1.27 1.27)
+				)
+				(justify left)
+			)
+		)
+		(property "Footprint" ""
+			(at 72.39 157.48 0)
+			(effects
+				(font
+					(size 1.27 1.27)
+				)
+				(hide yes)
+			)
+		)
+		(property "Datasheet" ""
+			(at 72.39 157.48 0)
+			(effects
+				(font
+					(size 1.27 1.27)
+				)
+				(hide yes)
+			)
+		)
+		(property "Description" ""
+			(at 72.39 157.48 0)
+			(effects
+				(font
+					(size 1.27 1.27)
+				)
+				(hide yes)
+			)
+		)
+		(pin "1"
+		)
+		(instances
+			(project "cover_flex"
+				(path "/b53ed5b7-46c8-5996-a3fb-579e9f592242"
+					(reference "#PWR013")
+					(unit 1)
+				)
+			)
+		)
+	)
+	(symbol
+		(lib_id "sensor:+5V")
+		(at 80.01 157.48 0)
+		(unit 1)
+		(exclude_from_sim no)
+		(in_bom no)
+		(on_board no)
+		(dnp no)
+		(property "Reference" "#PWR014"
+			(at 83.01 149.48 0)
+			(effects
+				(font
+					(size 1.27 1.27)
+				)
+				(justify left)
+				(hide yes)
+			)
+		)
+		(property "Value" "+5V"
+			(at 83.01 165.98 0)
+			(effects
+				(font
+					(size 1.27 1.27)
+				)
+				(justify left)
+			)
+		)
+		(property "Footprint" ""
+			(at 80.01 157.48 0)
+			(effects
+				(font
+					(size 1.27 1.27)
+				)
+				(hide yes)
+			)
+		)
+		(property "Datasheet" ""
+			(at 80.01 157.48 0)
+			(effects
+				(font
+					(size 1.27 1.27)
+				)
+				(hide yes)
+			)
+		)
+		(property "Description" ""
+			(at 80.01 157.48 0)
+			(effects
+				(font
+					(size 1.27 1.27)
+				)
+				(hide yes)
+			)
+		)
+		(pin "1"
+		)
+		(instances
+			(project "cover_flex"
+				(path "/b53ed5b7-46c8-5996-a3fb-579e9f592242"
+					(reference "#PWR014")
+					(unit 1)
+				)
+			)
+		)
+	)
+	(symbol
 		(lib_id "sensor:PWR_FLAG")
 		(at 35.56 50.8 0)
@@
 		(on_board no)
 		(dnp no)
-		(property "Reference" "#PWR013"
+		(property "Reference" "#PWR015"
 			(at 38.56 42.8 0)
 			(effects
@@
 			(project "cover_flex"
 				(path "/b53ed5b7-46c8-5996-a3fb-579e9f592242"
-					(reference "#PWR013")
+					(reference "#PWR015")
 					(unit 1)
 				)
@@
 		(on_board no)
 		(dnp no)
-		(property "Reference" "#PWR014"
+		(property "Reference" "#PWR016"
 			(at 69.04 42.8 0)
 			(effects
@@
 			(project "cover_flex"
 				(path "/b53ed5b7-46c8-5996-a3fb-579e9f592242"
-					(reference "#PWR014")
-					(unit 1)
-				)
+					(reference "#PWR016")
+					(unit 1)
+				)
