File: pcb/sensor/kicad/eu_cap_board.kicad_pcb (KiCad board)
At the start: 2 copper layers, 76 x 113.8 mm, 20 parts, among them J2 55909-2474, U1 SHT40, U2 ADAU7002

Commit message: Version v0.6 (D-120): boards, fab and PCBWay packs, order upload name and renders renamed; v0.5 files removed
Other:
- board text added: "EU CAP BOARD v0.6 (D-70)"
- board text removed: "EU CAP BOARD v0.5 (D-70)"
