File: pcb/sensor/kicad/ring_board.kicad_pcb (KiCad board)
At the start: 2 copper layers, 66.3 x 125.8 mm, 15 parts, among them J1 5V in (FFC), J2 55909-2474, U1 SHT40, U2 ADAU7002

Commit message: Version v0.6 (D-120): boards, fab and PCBWay packs, order upload name and renders renamed; v0.5 files removed
Other:
- board text added: "RING BOARD v0.6 (D-50)"
- board text removed: "RING BOARD v0.5 (D-50)"
