File: pcb/sensor/kicad/riser_board.kicad_sch (KiCad schematic)
At the start: 4 parts, among them J1 +5V pin, J2 GND pin, P1 +5V post, P2 GND post

Commit message: Flex review fixes, back cover clip, README, Sladdseg, order lists (D-116..D-119)
- D-116: cover flex: 0603 X5R input/output caps, ESD diode TPD1E10B06DYAR,
  0.6 mm bend radius with relief slits, stiffener notch and outlines,
  coverlay expansion, mask-defined pin pads, teardrops, fab notes; the
  cover's snap hooks allow for stiffener adhesive and tolerance
- D-117, D-118: bottom clip catch 3.22 above the floor, tip as far proud of
  the shell as the top clip's
- Battery polarity confirmed on a unit
- README rewritten: three editions, assembly renders, safety and polarity
  warnings, cost for 1 to 10,000 plates, printed parts; detail and board
  renders moved to their docs; the product is named Sladdseg
- EU boards: the ant logo on the other face
- D-119: order lists: one NA plate, one EU plate, a devkit of 5 + 5
Other:
- title: Smart wall plate - riser board -> Sladdseg - riser board
Changed lines of the file:
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@@
 	(paper "A4")
 	(title_block
-		(title "Smart wall plate - riser board")
+		(title "Sladdseg - riser board")
 		(date "2026-10-12")
 		(rev "v0.5")
