File: pcb/eu/kicad/eu_5v_board.kicad_pcb (KiCad board)
At the start: 2 copper layers, 57.9 x 27.9 mm, 10 parts, among them J1 Socket 1x2 2.54, P1 P70-2200045 GND, P2 P70-2200045 +5V, P3 P70-2200045 +5V, P4 P70-2200045 GND

Commit message: Flex review fixes, back cover clip, README, Sladdseg, order lists (D-116..D-119)
- D-116: cover flex: 0603 X5R input/output caps, ESD diode TPD1E10B06DYAR,
  0.6 mm bend radius with relief slits, stiffener notch and outlines,
  coverlay expansion, mask-defined pin pads, teardrops, fab notes; the
  cover's snap hooks allow for stiffener adhesive and tolerance
- D-117, D-118: bottom clip catch 3.22 above the floor, tip as far proud of
  the shell as the top clip's
- Battery polarity confirmed on a unit
- README rewritten: three editions, assembly renders, safety and polarity
  warnings, cost for 1 to 10,000 plates, printed parts; detail and board
  renders moved to their docs; the product is named Sladdseg
- EU boards: the ant logo on the other face
- D-119: order lists: one NA plate, one EU plate, a devkit of 5 + 5
Parts:
- LOGO1: moved to F.Cu
- turned LOGO1 to 0 degrees

Commit message: Version v0.6 (D-120): boards, fab and PCBWay packs, order upload name and renders renamed; v0.5 files removed
Other:
- board text added: "EU 5V v0.6"
- board text removed: "EU 5V v0.5"
