File: pcb/eu/kicad/eu_mains_board.kicad_pcb (KiCad board)
At the start: 2 copper layers, 57.9 x 57.9 mm, 12 parts, among them J1 2604-3102, J2 2604-3102, J3 TSM-102-02-L-SV

Commit message: Flex review fixes, back cover clip, README, Sladdseg, order lists (D-116..D-119)
- D-116: cover flex: 0603 X5R input/output caps, ESD diode TPD1E10B06DYAR,
  0.6 mm bend radius with relief slits, stiffener notch and outlines,
  coverlay expansion, mask-defined pin pads, teardrops, fab notes; the
  cover's snap hooks allow for stiffener adhesive and tolerance
- D-117, D-118: bottom clip catch 3.22 above the floor, tip as far proud of
  the shell as the top clip's
- Battery polarity confirmed on a unit
- README rewritten: three editions, assembly renders, safety and polarity
  warnings, cost for 1 to 10,000 plates, printed parts; detail and board
  renders moved to their docs; the product is named Sladdseg
- EU boards: the ant logo on the other face
- D-119: order lists: one NA plate, one EU plate, a devkit of 5 + 5
Parts:
- LOGO1: moved to B.Cu
- turned LOGO1 to 180 degrees

Commit message: Variants equal: na/eu/shared layout, shared part names, no default variant (D-125)
Parts:
- F1: footprint eu:Fuse_Schurter_UMT250 -> eu_mains:Fuse_Schurter_UMT250
- J1, J2: footprint eu:WAGO_2604-3102_1x02_P5.00mm_Vertical -> eu_mains:WAGO_2604-3102_1x02_P5.00mm_Vertical
- J3: footprint eu:PinHeader_1x02_P2.54mm_Vertical_SMD_Pin1Left -> eu_mains:PinHeader_1x02_P2.54mm_Vertical_SMD_Pin1Left
- LOGO1: footprint eu:Ant_Logo_8mm_SilkScreen -> eu_mains:Ant_Logo_8mm_SilkScreen
- LOGO2: footprint eu:KiCad-Logo2_5mm_SilkScreen -> eu_mains:KiCad-Logo2_5mm_SilkScreen
- MH1, MH2, MH3: footprint eu:MountingHole_2.2mm_M2 -> eu_mains:MountingHole_2.2mm_M2
- PS1: footprint eu:Converter_ACDC_Zettler_ZPI03_THT -> eu_mains:Converter_ACDC_Zettler_ZPI03_THT
- RV1: footprint eu:Varistor_TDK_CU4032 -> eu_mains:Varistor_TDK_CU4032
- S1: footprint eu:Rocker_DPST_Marquardt_1802.2504_E-Switch_RA412C1100 -> eu_mains:Rocker_DPST_Marquardt_1802.2504_E-Switch_RA412C1100

Commit message: v0.6: one barrier per variant, EU ridges, NA cable slit, ElegooSlicer projects, back cover and plate fixes (D-127..D-150)
- One barrier per variant for every edition; printed blank board in switch only (D-127..D-131)
- EU pin board ridge loop and blank board ridge; more pin board bosses (D-128..D-133)
- NA face plate lobes round the screws form the pocket's ends (D-132)
- NA 5 V cable straight from J2 to J1 through a slit in the barrier's bottom wall, 50 mm FFC; MH3 back in line;
  slit open in battery-free and switch only (D-134, D-135)
- Back cover: flex pad section 1.5 mm in, rim cut at the bottom end with a 0.08 mm-layer taper, steel plate clips
  solid in the shell, bottom clip lead-in 45 deg, pry notch 1.5 deep (D-136..D-143, D-145, D-147)
- 45 deg chamfer round the remote pocket's mouth (D-139)
- Print projects built with ElegooSlicer 1.5.3.5, overrides also as object settings (D-144)
- EU plain face plate 84.6 x 84.6, plain carrier whole on all sides with the full rim (D-146, D-150)
- Steel piece 1.0 mm thick, recess 1.2 deep (D-148)
- MSR-2 12 mm left, grille on the plate's centre line; ant logos in the sensor boards' lower-left corners (D-149)
- Repo URL github.com/antevens/sladdseg on the boards
Other:
- board text added: "github.com/antevens/sladdseg"
- board text removed: "github.com/antevens/smart-wallplate"
