File: pcb/eu/kicad/eu_sensor_board.kicad_pcb (KiCad board)
At the start: 2 copper layers, 76 x 113.8 mm, 20 parts, among them J2 55909-2474, U1 SHT40, U2 ADAU7002

Commit message: v0.6: one barrier per variant, EU ridges, NA cable slit, ElegooSlicer projects, back cover and plate fixes (D-127..D-150)
- One barrier per variant for every edition; printed blank board in switch only (D-127..D-131)
- EU pin board ridge loop and blank board ridge; more pin board bosses (D-128..D-133)
- NA face plate lobes round the screws form the pocket's ends (D-132)
- NA 5 V cable straight from J2 to J1 through a slit in the barrier's bottom wall, 50 mm FFC; MH3 back in line;
  slit open in battery-free and switch only (D-134, D-135)
- Back cover: flex pad section 1.5 mm in, rim cut at the bottom end with a 0.08 mm-layer taper, steel plate clips
  solid in the shell, bottom clip lead-in 45 deg, pry notch 1.5 deep (D-136..D-143, D-145, D-147)
- 45 deg chamfer round the remote pocket's mouth (D-139)
- Print projects built with ElegooSlicer 1.5.3.5, overrides also as object settings (D-144)
- EU plain face plate 84.6 x 84.6, plain carrier whole on all sides with the full rim (D-146, D-150)
- Steel piece 1.0 mm thick, recess 1.2 deep (D-148)
- MSR-2 12 mm left, grille on the plate's centre line; ant logos in the sensor boards' lower-left corners (D-149)
- Repo URL github.com/antevens/sladdseg on the boards
Parts:
- moved LOGO1 102.4 mm to (69.0, 143.5)
- moved C3 12.0 mm to (123.5, 57.3)
- moved C4 12.0 mm to (114.8, 55.9)
- moved H1 12.0 mm to (68.0, 64.0)
- moved H5 12.0 mm to (78.2, 51.7)
- moved H6 12.0 mm to (94.3, 51.7)
- moved H7 12.0 mm to (70.5, 46.3)
- moved J2 12.0 mm to (100.6, 47.8)
- moved MK1 12.0 mm to (120.0, 55.8)
- moved R1 12.0 mm to (112.5, 55.4)
- moved U2 12.0 mm to (115.9, 55.0)
Routing:
- net +3V3: track 220.3 -> 208.3 mm
- net /SDA: track 175.0 -> 163.0 mm
- net /SCL: track 176.1 -> 164.1 mm
- net +5V: track 102.4 -> 114.4 mm
Other:
- outline, holes or cut-outs redrawn
- board text added: "github.com/antevens/sladdseg"
- board text removed: "github.com/antevens/smart-wallplate"

Commit message: Version v0.7 (D-151): boards, fab and PCBWay packs, order upload name and section renders renamed; v0.6 files removed
Other:
- board text added: "EU SENSOR BOARD v0.7 (D-70)"
- board text removed: "EU SENSOR BOARD v0.6 (D-70)"
