File: pcb/kicad/wiring_board.kicad_pcb (KiCad board)
At the start: 2 copper layers, 47 x 72 mm, 14 parts, among them J1 2604-1106, J2 5V out (FFC to the ring board), P1 +5V post, P2 GND post

Commit message: Version v0.6 (D-120): boards, fab and PCBWay packs, order upload name and renders renamed; v0.5 files removed
Other:
- board text added: "wiring_board v0.6"
- board text removed: "wiring_board v0.5"
