File: pcb/na/kicad/na_mains_board.kicad_pcb (KiCad board)
At the start: 2 copper layers, 47 x 72 mm, 14 parts, among them J1 2604-1106, J2 5V out (FFC to the sensor boa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, P1 +5V post, P2 GND post

Commit message: v0.6: one barrier per variant, EU ridges, NA cable slit, ElegooSlicer projects, back cover and plate fixes (D-127..D-150)
- One barrier per variant for every edition; printed blank board in switch only (D-127..D-131)
- EU pin board ridge loop and blank board ridge; more pin board bosses (D-128..D-133)
- NA face plate lobes round the screws form the pocket's ends (D-132)
- NA 5 V cable straight from J2 to J1 through a slit in the barrier's bottom wall, 50 mm FFC; MH3 back in line;
  slit open in battery-free and switch only (D-134, D-135)
- Back cover: flex pad section 1.5 mm in, rim cut at the bottom end with a 0.08 mm-layer taper, steel plate clips
  solid in the shell, bottom clip lead-in 45 deg, pry notch 1.5 deep (D-136..D-143, D-145, D-147)
- 45 deg chamfer round the remote pocket's mouth (D-139)
- Print projects built with ElegooSlicer 1.5.3.5, overrides also as object settings (D-144)
- EU plain face plate 84.6 x 84.6, plain carrier whole on all sides with the full rim (D-146, D-150)
- Steel piece 1.0 mm thick, recess 1.2 deep (D-148)
- MSR-2 12 mm left, grille on the plate's centre line; ant logos in the sensor boards' lower-left corners (D-149)
- Repo URL github.com/antevens/sladdseg on the boards
Parts:
- moved MH3 8.73 mm to (121.0, 66.5)
- moved J2 1.70 mm to (112.7, 123.3), turned to 0 degrees
Routing:
- net +5V: track 20.1 -> 26.7 mm
Other:
- board text added: "FFC ↓ TO THE SLOT"
- board text added: "THIS SIDE"
- board text added: "TO THE ROOM"
- board text added: "github.com/antevens/sladdseg"
- board text added: "↑ UP"
- board text added: "↑ UP THIS SIDE INTO THE BOX"
- board text removed: "github.com/antevens/smart-wallplate"

Commit message: Version v0.7 (D-151): boards, fab and PCBWay packs, order upload name and section renders renamed; v0.6 files removed
Other:
- board text added: "2026-10-13"
- board text added: "NA MAINS v0.7"
- board text removed: "2026-10-12"
- board text removed: "NA MAINS v0.6"
