File: pcb/na/kicad/na_mains_board.kicad_sch (KiCad schematic)
At the start: 8 parts, among them J1 2604-1106, J2 5V out (FFC to the sensor boa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, P1 +5V post, P2 GND post

Commit message: v0.6: one barrier per variant, EU ridges, NA cable slit, ElegooSlicer projects, back cover and plate fixes (D-127..D-150)
- One barrier per variant for every edition; printed blank board in switch only (D-127..D-131)
- EU pin board ridge loop and blank board ridge; more pin board bosses (D-128..D-133)
- NA face plate lobes round the screws form the pocket's ends (D-132)
- NA 5 V cable straight from J2 to J1 through a slit in the barrier's bottom wall, 50 mm FFC; MH3 back in line;
  slit open in battery-free and switch only (D-134, D-135)
- Back cover: flex pad section 1.5 mm in, rim cut at the bottom end with a 0.08 mm-layer taper, steel plate clips
  solid in the shell, bottom clip lead-in 45 deg, pry notch 1.5 deep (D-136..D-143, D-145, D-147)
- 45 deg chamfer round the remote pocket's mouth (D-139)
- Print projects built with ElegooSlicer 1.5.3.5, overrides also as object settings (D-144)
- EU plain face plate 84.6 x 84.6, plain carrier whole on all sides with the full rim (D-146, D-150)
- Steel piece 1.0 mm thick, recess 1.2 deep (D-148)
- MSR-2 12 mm left, grille on the plate's centre line; ant logos in the sensor boards' lower-left corners (D-149)
- Repo URL github.com/antevens/sladdseg on the boards
Other:
- company: smart-wallplate -> sladdseg
Changed lines of the file:
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@@
 		(date "2026-10-12")
 		(rev "v0.6")
-		(company "smart-wallplate")
+		(company "sladdseg")
 		(comment 1 "Spacing values are design targets - human review before fab.")
 		(comment 2 "Generated by pcb/na/tools/gen_schematic_na.py - edit parts_na.py")
